File: pickit4_adapter/pickit4_adapter.brd (EAGLE design)
At the start: 26.7 x 22.9 mm, 15 parts, among them J1 TSW-108-16-L-S-RA, J2 ZX62R-B-5P(30), J3 TSW-106-16-L-S-RA, U1 STLQ015M33R, U2 MCP2221AT-I/ST

Commit message: refactor: fixed ignored files and added tables
Parts:
- added FID1, FID2, FID3: FIDUCIAL_1MM_TOP_BOTTOM, HatchPoint:FIDUCIAL_1MM_TOP_BOTTOM
Changed lines of the file:
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@@
 <layer number="56" name="wert" color="7" fill="1" visible="no" active="no"/>
 <layer number="57" name="tCAD" color="7" fill="1" visible="no" active="no"/>
+<layer number="58" name="bCAD" color="7" fill="1" visible="no" active="no"/>
 <layer number="59" name="tCarbon" color="7" fill="1" visible="no" active="no"/>
 <layer number="60" name="bCarbon" color="7" fill="1" visible="no" active="no"/>
@@
 </attributes>
 <variantdefs>
+<variantdef name="A"/>
 </variantdefs>
 <classes>
@@
 <attribute name="VDC" value="25V" x="6.6675" y="13.6525" size="1.778" layer="27" display="off"/>
 </element>
+<element name="FID1" library="HatchPoint" package="FIDUCIAL_1MM_TOP_BOTTOM" value="FIDUCIAL_1MM_TOP_BOTTOM" x="3.81" y="2.54" smashed="yes"/>
+<element name="FID2" library="HatchPoint" package="FIDUCIAL_1MM_TOP_BOTTOM" value="FIDUCIAL_1MM_TOP_BOTTOM" x="3.81" y="20.32" smashed="yes"/>
+<element name="FID3" library="HatchPoint" package="FIDUCIAL_1MM_TOP_BOTTOM" value="FIDUCIAL_1MM_TOP_BOTTOM" x="20.32" y="5.08" smashed="yes"/>
 </elements>
 <signals>
