File: pickit4_adapter/pickit4_adapter.sch (EAGLE design)
At the start: 15 parts, among them J1 TSW-108-16-L-S-RA, J2 ZX62R-B-5P(30), J3 TSW-106-16-L-S-RA, U1 STLQ015M33R, U2 MCP2221AT-I/ST

Commit message: refactor: fixed ignored files and added tables
Parts:
- added FID1, FID2, FID3: FIDUCIAL_1MM_TOP_BOTTOM, HatchPoint:FIDUCIAL_1MM_TOP_BOTTOM
Other:
- note added: "01/30/2022"
- note added: "Document creation."
- note added: "R1,0"
- note added: "RSL"
Changed lines of the file:
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@@
 <layer number="56" name="wert" color="7" fill="1" visible="no" active="no"/>
 <layer number="57" name="tCAD" color="7" fill="1" visible="no" active="no"/>
+<layer number="58" name="bCAD" color="7" fill="1" visible="no" active="no"/>
 <layer number="59" name="tCarbon" color="7" fill="1" visible="no" active="no"/>
 <layer number="60" name="bCarbon" color="7" fill="1" visible="no" active="no"/>
@@
 <schematic xreflabel="%F%N/%S.%C%R" xrefpart="/%S.%C%R">
 <attributes>
+<attribute name="APPROVED" value="MK"/>
 <attribute name="CONTACT" value="rluttrell@hatchpoint.com (901)605-3388"/>
+<attribute name="CREATED_DATE_TIME" value="01/30/2022 3:31 PM"/>
 <attribute name="DESIGNED" value="RSL"/>
 <attribute name="FILENAME" value="PICKIT4_Programming_Board.sch"/>
 <attribute name="REV" value="1.0"/>
-<attribute name="SCHEMATIC_TITLE" value="PICkit4 Programming Board"/>
+<attribute name="SCHEMATIC_TITLE" value="PICkit4 Adapter Board"/>
 <attribute name="SIZE" value="LET"/>
 </attributes>
 <variantdefs>
+<variantdef name="A"/>
 </variantdefs>
 <classes>
@@
 </classes>
 <parts>
-<part name="FRAME1" library="HatchPoint-Frames" library_urn="urn:adsk.eagle:library:5099271" deviceset="FRAME_A_L_VER2" device="">
-<attribute name="CONTACT" value=""/>
-<attribute name="DESIGNED" value=""/>
-<attribute name="FILENAME" value=""/>
-<attribute name="REV" value=""/>
-<attribute name="SCHEMATIC_TITLE" value=""/>
-<attribute name="SIZE" value=""/>
-</part>
-<part name="FRAME2" library="HatchPoint-Frames" library_urn="urn:adsk.eagle:library:5099271" deviceset="FRAME_A_L_VER2" device="">
-<attribute name="CONTACT" value=""/>
-<attribute name="DESIGNED" value=""/>
-<attribute name="FILENAME" value=""/>
-<attribute name="REV" value=""/>
-<attribute name="SCHEMATIC_TITLE" value=""/>
-<attribute name="SIZE" value=""/>
-</part>
 <part name="U2" library="HatchPoint-MicrochipTechnology" library_urn="urn:adsk.eagle:library:24060010" deviceset="MCP2221AT-*" device="I/ST" package3d_urn="urn:adsk.eagle:package:31336517/2"/>
 <part name="FL1" library="HatchPoint-ST" library_urn="urn:adsk.eagle:library:23797591" deviceset="USBDF0*W5" device="" package3d_urn="urn:adsk.eagle:package:27499786/2" technology="1"/>
@@
 <part name="V4" library="HatchPoint-Supplies" library_urn="urn:adsk.eagle:library:8624175" deviceset="+3V3" device=""/>
 <part name="GND5" library="HatchPoint-Supplies" library_urn="urn:adsk.eagle:library:8624175" deviceset="DGND" device=""/>
+<part name="FRAME1" library="HatchPoint-Frames" library_urn="urn:adsk.eagle:library:5099271" deviceset="FRAME_A_L_VER2" device="">
+<attribute name="APPROVED" value=""/>
+<attribute name="CREATED_DATE_TIME" value=""/>
+</part>
+<part name="FRAME2" library="HatchPoint-Frames" library_urn="urn:adsk.eagle:library:5099271" deviceset="FRAME_A_L_VER2" device=""/>
+<part name="FID1" library="HatchPoint" deviceset="FIDUCIAL" device="_1MM_TOP_BOTTOM">
+<variant name="A" populate="no"/>
+</part>
+<part name="FID2" library="HatchPoint" deviceset="FIDUCIAL" device="_1MM_TOP_BOTTOM">
+<variant name="A" populate="no"/>
+</part>
+<part name="FID3" library="HatchPoint" deviceset="FIDUCIAL" device="_1MM_TOP_BOTTOM">
+<variant name="A" populate="no"/>
+</part>
+<part name="TBL1" library="HatchPoint-Frames" library_urn="urn:adsk.eagle:library:5099271" deviceset="REVISION_TABLE" device=""/>
 </parts>
 <sheets>
 <sheet>
-<description>Interface</description>
+<description>Revision Table</description>
 <plain>
+<text x="10.16" y="187.96" size="2.54" layer="94">01/30/2022</text>
+<text x="30.48" y="187.96" size="2.54" layer="94">RSL</text>
+<text x="45.72" y="187.96" size="2.54" layer="94">R1,0</text>
+<text x="60.96" y="187.96" size="2.54" layer="94">Document creation.</text>
 </plain>
 <instances>
 <instance part="FRAME2" gate="G$1" x="0" y="0" smashed="yes"/>
 <instance part="FRAME2" gate="G$2" x="158.75" y="3.81" smashed="yes">
+<attribute name="CREATED_DATE_TIME" x="201.93" y="4.445" size="1.27" layer="94"/>
 <attribute name="SHEET" x="186.69" y="11.43" size="1.905" layer="94"/>
+<attribute name="SCHEMATIC_TITLE" x="201.93" y="39.37" size="3.81" layer="94"/>
+<attribute name="REV" x="171.45" y="11.43" size="1.905" layer="94"/>
+<attribute name="APPROVED" x="181.61" y="21.59" size="1.905" layer="94"/>
 <attribute name="SHEET_HEADLINE" x="201.93" y="26.67" size="2.54" layer="94"/>
+<attribute name="FILENAME" x="201.93" y="10.16" size="2.54" layer="94"/>
 <attribute name="LAST_DATE_TIME" x="240.03" y="4.445" size="1.27" layer="94"/>
-<attribute name="SCHEMATIC_TITLE" x="201.93" y="39.37" size="3.81" layer="94"/>
 <attribute name="DESIGNED" x="161.29" y="21.59" size="1.905" layer="94"/>
 <attribute name="SIZE" x="161.29" y="11.43" size="1.905" layer="94"/>
 <attribute name="CONTACT" x="161.29" y="4.445" size="1.27" layer="94"/>
-<attribute name="REV" x="171.45" y="11.43" size="1.905" layer="94"/>
-<attribute name="FILENAME" x="201.93" y="10.16" size="2.54" layer="94"/>
-</instance>
+</instance>
+<instance part="FID1" gate="G$1" x="172.72" y="76.2" smashed="yes"/>
+<instance part="FID2" gate="G$1" x="185.42" y="76.2" smashed="yes"/>
+<instance part="FID3" gate="G$1" x="198.12" y="76.2" smashed="yes"/>
+<instance part="TBL1" gate="G$1" x="7.62" y="193.04" smashed="yes"/>
 </instances>
 <busses>
@@
 </sheet>
 <sheet>
-<description>Revision Table</description>
+<description>Adapter Board</description>
 <plain>
 </plain>
 <instances>
-<instance part="FRAME1" gate="G$1" x="0" y="0" smashed="yes"/>
-<instance part="FRAME1" gate="G$2" x="158.75" y="3.81" smashed="yes">
-<attribute name="SHEET" x="186.69" y="11.43" size="1.905" layer="94"/>
-<attribute name="SHEET_HEADLINE" x="201.93" y="26.67" size="2.54" layer="94"/>
-<attribute name="LAST_DATE_TIME" x="240.03" y="4.445" size="1.27" layer="94"/>
-<attribute name="SCHEMATIC_TITLE" x="201.93" y="39.37" size="3.81" layer="94"/>
-<attribute name="DESIGNED" x="161.29" y="21.59" size="1.905" layer="94"/>
-<attribute name="SIZE" x="161.29" y="11.43" size="1.905" layer="94"/>
-<attribute name="CONTACT" x="161.29" y="4.445" size="1.27" layer="94"/>
-<attribute name="REV" x="171.45" y="11.43" size="1.905" layer="94"/>
-<attribute name="FILENAME" x="201.93" y="10.16" size="2.54" layer="94"/>
-</instance>
 <instance part="U2" gate="G$1" x="121.92" y="114.3" smashed="yes">
 <attribute name="NAME" x="127" y="121.92" size="1.778" layer="95"/>
@@
 </instance>
 <instance part="GND5" gate="G$1" x="71.12" y="170.18" smashed="yes"/>
+<instance part="FRAME1" gate="G$1" x="0" y="0" smashed="yes"/>
+<instance part="FRAME1" gate="G$2" x="158.75" y="3.81" smashed="yes">
+<attribute name="SHEET" x="186.69" y="11.43" size="1.905" layer="94"/>
+<attribute name="SCHEMATIC_TITLE" x="201.93" y="39.37" size="3.81" layer="94"/>
+<attribute name="REV" x="171.45" y="11.43" size="1.905" layer="94"/>
+<attribute name="SHEET_HEADLINE" x="201.93" y="26.67" size="2.54" layer="94"/>
+<attribute name="FILENAME" x="201.93" y="10.16" size="2.54" layer="94"/>
+<attribute name="LAST_DATE_TIME" x="240.03" y="4.445" size="1.27" layer="94"/>
+<attribute name="DESIGNED" x="161.29" y="21.59" size="1.905" layer="94"/>
+<attribute name="SIZE" x="161.29" y="11.43" size="1.905" layer="94"/>
+<attribute name="CONTACT" x="161.29" y="4.445" size="1.27" layer="94"/>
+<attribute name="APPROVED" x="181.61" y="21.59" size="1.905" layer="94"/>
+<attribute name="CREATED_DATE_TIME" x="201.93" y="4.445" size="1.27" layer="94"/>
+</instance>
 </instances>
 <busses>
